File: betrayal_char_counter.sch (KiCad schematic (older format))
At the start: 20 parts, among them J1 AVR-ISP-6, SW1 SW_ON, SW10 SW_Push, SW2 SW_Push, SW3 SW_Push, SW4 SW_Push, SW5 SW_Push, SW6 SW_Push, SW7 SW_Push, SW8 SW_Push, SW9 SW_Push, U1 MCP1640CH, U2 ATtiny88-AU

Commit message: Add 1mm height
Parts:
- BT1: value 3xAAA -> 1xAAA; footprint Battery:BatteryHolder_Keystone_2479_3xAAA -> Battery:BatteryHolder_Keystone_2466_1xAAA
Changed lines of the file:
@@
 P 5500 1650
 F 0 "BT1" H 5618 1746 50  0000 L CNN
-F 1 "3xAAA" H 5618 1655 50  0000 L CNN
-F 2 "Battery:BatteryHolder_Keystone_2479_3xAAA" V 5500 1710 50  0001 C CNN
+F 1 "1xAAA" H 5618 1655 50  0000 L CNN
+F 2 "Battery:BatteryHolder_Keystone_2466_1xAAA" V 5500 1710 50  0001 C CNN
 F 3 "~" V 5500 1710 50  0001 C CNN
 	1    5500 1650
